File: Teensy4.1-example.kicad_sch (KiCad schematic)
At the start: 80 parts, among them IC1 MIMXRT1062DVJ6B, J1 Conn_01x11_Male, J2 Conn_01x11_Male, J3 Conn_01x12_Male, J4 Conn_01x11_Male, J5 Conn_01x11_Male, J6 Conn_01x03_Male, J7 Conn_01x03_Male, P2 D26, Q1 Q_PMOS_GDS_DMP3125L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

Commit message: add phy chip to schematic
Parts:
- added C?: 0.22uf, Capacitor_SMD:C_0603_1608Metric, symbol Device:C
- added C?: 2.2uf, Capacitor_SMD:C_0603_1608Metric, symbol Device:C
- added C?: 10nf, Capacitor_SMD:C_0603_1608Metric, symbol Device:C
- added U5: DP83825IRMQR, XCVR_DP83825IRMQR, symbol DP83825IRMQR:DP83825IRMQR
Connections:
- net +3V3: now also C?.1, C?.1, C?.1, U5.19 (VDDIO), U5.6 (VDDA3V3)
- net GND: now also C?.2, C?.2, C?.2
- net TXD1: now reaches IC1.A12 (GPIO_B1_08)
- net TXD1: now also U5.24 (TX_D1)
- net TXEN: now reaches IC1.A13 (GPIO_B1_09)
- net TXEN: now also U5.1 (TX_EN)
- net TXD0: now reaches IC1.B12 (GPIO_B1_07)
- net TXD0: now also U5.23 (TX_D0)
- net XI: now reaches IC1.B13 (GPIO_B1_10)
- net XI: now also U5.13 (XI/50MHZIN)
- net MDIO: now reaches IC1.B14 (GPIO_B1_15)
- net MDIO: now also U5.15 (MDIO)
- net DV: now reaches IC1.C12 (GPIO_B1_06)
- net DV: now also U5.2 (50MHZOUT/LED2/S(RX_DV_EN))
- net RXER: now reaches IC1.C13 (GPIO_B1_11)
- net RXER: now also U5.22 (RX_ER/S(A-MDIX))
- net MDC: now reaches IC1.C14 (GPIO_B1_14)
- net MDC: now also U5.16 (MDC)
- net RXD1: now reaches IC1.D12 (GPIO_B1_05)
- net RXD1: now also U5.17 (RX_D1/S(MASTER/SLAVE))
- net RST: now reaches IC1.E10 (GPIO_B0_14)
- net RST: now also U5.5 (~{RST})
- net INT: now reaches IC1.E11 (GPIO_B0_15)
- net INT: now also U5.3 (INTR/PWRDN)
- net RXD0: now reaches IC1.E12 (GPIO_B1_04)
- net RXD0: now also U5.18 (RX_D0/S(PHYADD0))
- no-connect marks 66 -> 54

Commit message: add ARJP11B magjack
Parts:
- removed D2: LED, LED_SMD:LED_0402_1005Metric, symbol Device:LED
- removed Di3: SP0503BAHT, Package_TO_SOT_SMD:SOT-143, symbol Power_Protection:SP0503BAHT
- removed R12, R13: 56k, Resistor_SMD:R_0603_1608Metric, symbol Device:R
- removed R16: 100k, Resistor_SMD:R_0603_1608Metric, symbol Device:R
- removed R6, R7: 16k, Resistor_SMD:R_0603_1608Metric, symbol Device:R
- removed R8: 1k, Resistor_SMD:R_0402_1005Metric, symbol Device:R
- removed R9: 1M, Resistor_SMD:R_0603_1608Metric, symbol Device:R
- removed U2: MAX1562, Package_SO:SO-8_3.9x4.9mm_P1.27mm, symbol MIMXRT1062DVJ6B:MAX1562
- removed USB_DFP1: USB_C_Receptacle_USB2.0, USB-C-Power-tester:TYPE-C-31-M-14, symbol simonsen:USB_C_Receptacle_USB2.0_NOPOW
- added J8: ARJP11B-MASA-B-A-EMU2, ARJP11B-MASA-B-A-EMU2:ARJP11B-MASA-B-A-EMU2, symbol ARJP11B-MASA-B-A-EMU2:ARJP11B-MASA-B-A-EMU2
- added R17: 150, Resistor_SMD:R_0603_1608Metric, symbol Device:R
- added R18: 6.49K, Resistor_SMD:R_0603_1608Metric, symbol Device:R
- U5: footprint XCVR_DP83825IRMQR -> DP83825IRMQR:XCVR_DP83825IRMQR
- gave numbers to parts that had none: 3
Connections:
- net GND: now also U5.21 (GND), U5.25 (EXP), U5.26 (EXP), U5.27 (EXP), U5.28 (EXP), U5.29 (EXP), U5.30 (EXP), U5.9 (GND), J8.12 (CATHODE), R18.2
- net T-: now reaches U5.10 (TD_M)
- net T-: now also J8.2 (TD-)
- net T+: now reaches U5.11 (TD_P)
- net T+: now also J8.1 (TD+)
- net at U5.14 (RBIAS): now also R18.1
- net at U5.4 (LED0/S(ANEG_DIS)): now also R17.2
- net R-: now reaches U5.7 (RD_M)
- net R-: now also J8.6 (RD-)
- net R+: now reaches U5.8 (RD_P)
- net R+: now also J8.3 (RD+)
- new net ACK_LED: J8.11 (ANODE), R17.1
- no-connect marks 54 -> 56
